Commit message: Manually tuning the camera transform

File: robots/common/franka_arm.xacro (robot description, xacro)
@@ -127,4 +127,10 @@
       <child link="${prefix}link8" />
     </joint>
+    <joint name="${prefix}camera_joint" type="fixed">
+      <parent link="${prefix}link1" />
+      <child link="camera_link" />
+      <origin xyz="0.06 0 -0.16" rpy="3.14159 0 0" />
+    </joint>
+    <link name="camera_link"/>
   </xacro:macro>
 </robot>

Commit message: Attach camera to table rather than fr_link1

File: robots/common/franka_arm.xacro (robot description, xacro)
@@ -128,7 +128,7 @@
     </joint>
     <joint name="${prefix}camera_joint" type="fixed">
-      <parent link="${prefix}link1" />
+      <parent link="base" />
       <child link="camera_link" />
-      <origin xyz="0.06 0 -0.16" rpy="3.14159 0 0" />
+      <origin xyz="0.05 1.11 0.6" rpy="0 0.2 -1.05" />
     </joint>
     <link name="camera_link"/>

Commit message: Add camera mount and ground plane to franka_arm.xacro

File: robots/common/franka_arm.xacro (robot description, xacro)
@@ -133,4 +133,66 @@
     </joint>
     <link name="camera_link"/>
+    <joint name="${prefix}camera_mount_joint" type="fixed">
+      <parent link="base" />
+      <child link="camera_mount" />
+      <origin xyz="-0.09 0.2 0.0" rpy="0 0 0" />
+    </joint>
+    <link name="camera_mount">
+      <visual>
+        <origin xyz="0 0 0.1" rpy="0 0 0"/>
+        <geometry>
+          <box size="0.2 0.2 0.2"/>
+        </geometry>
+        <material name="green">
+          <color rgba="0.0 1.0 0.0 1"/>
+        </material>
+      </visual>
+      <collision>
+        <origin xyz="0 -0.1 0" rpy="0 0 0"/>
+        <geometry>
+          <box size="0.2 0.2 0.2"/>
+        </geometry>
+      </collision>
+    </link>
+    <joint name="ground_plane_joint" type="fixed">
+      <parent link="base" />
+      <child link="ground_plane" />
+      <origin xyz="0 0 0.0" rpy="0 0 0" />
+    </joint>
+    <link name="ground_plane">
+      <visual>
+        <geometry>
+          <box size="1 1 0.01"/>
+        </geometry>
+        <material name="brown">
+          <color rgba="0.5 0.5 0.0 0.3"/>
+        </material>
+      </visual>
+      <collision>
+        <geometry>
+          <box size="1 1 0.01"/>
+        </geometry>
+      </collision>
+    </link>
+    <joint name="driver_box_joint" type="fixed">
+      <parent link="base" />
+      <child link="driver_box" />
+      <origin xyz="-0.32 0 0.045" rpy="0 0 0" />
+    </joint>
+    <link name="driver_box">
+      <visual>
+        <geometry>
+          <box size="0.36 0.44 0.09"/>
+        </geometry>
+        <material name="black">
+          <color rgba="0.0 0.0 0.0 0.3"/>
+        </material>
+      </visual>
+      <collision>
+        <geometry>
+          <box size="0.36 0.44 0.09"/>
+        </geometry>
+      </collision>
+    </link>
   </xacro:macro>
 </robot>

Commit message: Tweak collision plane location, camera locations in URDF

File: robots/common/franka_arm.xacro (robot description, xacro)
@@ -130,5 +130,5 @@
       <parent link="base" />
       <child link="camera_link" />
-      <origin xyz="0.05 1.11 0.6" rpy="0 0.2 -1.05" />
+      <origin xyz="0.00 0.195 0.22" rpy="0 0.524 -0.262" />
     </joint>
     <link name="camera_link"/>
@@ -136,5 +136,5 @@
       <parent link="base" />
       <child link="camera_mount" />
-      <origin xyz="-0.09 0.2 0.0" rpy="0 0 0" />
+      <origin xyz="-0.07 0.2 0.0" rpy="0 0 0" />
     </joint>
     <link name="camera_mount">
@@ -145,5 +145,5 @@
         </geometry>
         <material name="green">
-          <color rgba="0.0 1.0 0.0 1"/>
+          <color rgba="0.0 1.0 0.0 0.3"/>
         </material>
       </visual>
@@ -158,5 +158,5 @@
       <parent link="base" />
       <child link="ground_plane" />
-      <origin xyz="0 0 0.0" rpy="0 0 0" />
+      <origin xyz="0 0 0.06" rpy="0 0 0" />
     </joint>
     <link name="ground_plane">

Commit message: Tweak collision plane location, camera locations in URDF

File: robots/common/franka_arm.xacro (robot description, xacro)
@@ -140,5 +140,5 @@
     <link name="camera_mount">
       <visual>
-        <origin xyz="0 0 0.1" rpy="0 0 0"/>
+        <origin xyz="0 -0.1 0" rpy="0 0 0"/>
         <geometry>
           <box size="0.2 0.2 0.2"/>

Commit message: Tweak camera_link pose

File: robots/common/franka_arm.xacro (robot description, xacro)
@@ -130,5 +130,5 @@
       <parent link="base" />
       <child link="camera_link" />
-      <origin xyz="0.00 0.195 0.22" rpy="0 0.524 -0.262" />
+      <origin xyz="0.07 0.195 0.22" rpy="0 0.524 -0.262" />
     </joint>
     <link name="camera_link"/>

Commit message: Move the ground plane down slightly

File: robots/common/franka_arm.xacro (robot description, xacro)
@@ -130,5 +130,5 @@
       <parent link="base" />
       <child link="camera_link" />
-      <origin xyz="0.07 0.195 0.22" rpy="0 0.524 -0.262" />
+      <origin xyz="0.07 0.195 0.21" rpy="0 0.524 -0.262" />
     </joint>
     <link name="camera_link"/>
@@ -158,5 +158,5 @@
       <parent link="base" />
       <child link="ground_plane" />
-      <origin xyz="0 0 0.06" rpy="0 0 0" />
+      <origin xyz="0 0 0.04" rpy="0 0 0" />
     </joint>
     <link name="ground_plane">

Commit message: Update camera pose

File: robots/common/franka_arm.xacro (robot description, xacro)
@@ -130,5 +130,5 @@
       <parent link="base" />
       <child link="camera_link" />
-      <origin xyz="0.07 0.195 0.21" rpy="0 0.524 -0.262" />
+      <origin xyz="0.056 0.21 0.26" rpy="0.059 0.51 -0.262" />
     </joint>
     <link name="camera_link"/>
