Commit message: Rotate the tcp frame for better teleop

File: end_effectors/common/franka_hand.xacro (robot description, xacro)
@@ -23,5 +23,5 @@
     <link name="${ee_prefix}hand_tcp" />
     <joint name="${ee_prefix}hand_tcp_joint" type="fixed">
-      <origin xyz="${tcp_xyz}" rpy="${tcp_rpy}" />
+      <origin xyz="${tcp_xyz}" rpy="0.0 -1.571 0.0" />
       <parent link="${ee_prefix}hand" />
       <child link="${ee_prefix}hand_tcp" />

Commit message: A bit of tolerance on gripper joint limits

File: end_effectors/common/franka_hand.xacro (robot description, xacro)
@@ -109,5 +109,6 @@
       <origin xyz="0 0 0.0584" rpy="0 0 0" />
       <axis xyz="0 1 0" />
-      <limit effort="100" lower="0.0" upper="0.04" velocity="0.2" />
+      <!-- Nominally 0.0/0.04 limits, we add a bit of tolerance -->
+      <limit effort="100" lower="-0.01" upper="0.05" velocity="0.2" />
       <dynamics damping="0.3" />
     </joint>
@@ -117,5 +118,6 @@
       <origin xyz="0 0 0.0584" rpy="0 0 0" />
       <axis xyz="0 -1 0" />
-      <limit effort="100" lower="0.0" upper="0.04" velocity="0.2" />
+      <!-- Nominally 0.0/0.04 limits, we add a bit of tolerance -->
+      <limit effort="100" lower="-0.01" upper="0.05" velocity="0.2" />
       <mimic joint="${ee_prefix}finger_joint1" />
       <dynamics damping="0.3" />
